File: MCU Datalogger.kicad_sch (KiCad schematic)
At the start: 4 parts

Commit message: pcb set up
Parts:
- added BT1: Battery, Connector_PinHeader_2.54mm:PinHeader_1x02_P2.54mm_Vertical, symbol Device:Battery
- added C1, C4: 0.1uF, Capacitor_SMD:C_0805_2012Metric, symbol Device:C
- added C2, C3: 22pF, Capacitor_SMD:C_0805_2012Metric, symbol Device:C
- added C5: 100nF, Capacitor_SMD:C_0805_2012Metric, symbol Device:C_Polarized
- added D1, D2: LED, LED_SMD:LED_0805_2012Metric, symbol Device:LED
- added H1, H2, H3, H4: MountingHole, MountingHole:MountingHole_2.1mm, symbol Mechanical:MountingHole
- added R5, R7: 330, Resistor_SMD:R_0805_2012Metric, symbol Device:R
- added R6: 10K, Resistor_SMD:R_0805_2012Metric, symbol Device:R
- added U1, U3: 24LC1025, Package_SO:SOIC-8_5.3x5.3mm_P1.27mm, symbol Memory_EEPROM:24LC1025
- added U2: DS1337S, DS1337S:SOIC127P600X175-8N, symbol DS1337S:DS1337S
- added U4: ATMEGA328-AU, ATMEGA328-AU:QFP80P900X900X120-32N, symbol ATMEGA328-AU:ATMEGA328-AU
- added Y1: 32.768KHz, Crystal:Crystal_SMD_5032-2Pin_5.0x3.2mm_HandSoldering, symbol Device:Crystal
- added Y2: 16MHz, Crystal:Crystal_SMD_5032-2Pin_5.0x3.2mm_HandSoldering, symbol Device:Crystal
- R1, R2: value R -> 10K; footprint (none) -> Resistor_SMD:R_0805_2012Metric
- R3, R4: value R -> 4.7K; footprint (none) -> Resistor_SMD:R_0805_2012Metric
Connections:
- net Vcc: now reaches R2.1
- net Vcc: now also R1.1, R3.1, R4.1, C1.1, R6.2, U1.1 (A0), U1.2 (A1), U1.3 (A2), U1.8 (VCC), U2.8 (VCC), U3.1 (A0), U3.3 (A2), U3.8 (VCC)
- net at R2.2: now also U2.7 (SQW/~INT)
- net SDA: now reaches R4.2
- net SDA: now also U1.5 (SDA), U2.5 (SDA), U3.5 (SDA), U4.27 (PC4)
- net SCK: now reaches R3.2
- net SCK: now also D1.2 (A), U1.6 (SCL), U2.6 (SCL), U3.6 (SCL), U4.17 (PB5), U4.28 (PC5)
- net at R1.2: now also U2.3 (~{INTA})
- new net: U2.2 (X2), Y1.1
- new net: U2.1 (X1), Y1.2
- new net: C3.1, U4.8 (PB7), Y2.2
- new net: D2.1 (K), R7.1
- new net: D1.1 (K), R5.2
- new net: C2.2, U4.7 (PB6), Y2.1
- new net: BT1.1 (+), C5.1, D2.2 (A), U4.18 (AVCC), U4.4 (VCC), U4.6 (VCC)
- new net: C4.2, U4.20 (AREF)
- new net D2: U4.32 (PD2)
- new net D3: U4.1 (PD3)
- new net D4: U4.2 (PD4)
- new net D5: U4.9 (PD5)
- new net D6: U4.10 (PD6)
- new net D7: U4.11 (PD7)
- new net D8: U4.12 (PB0)
- new net GND: BT1.2 (-), C1.2, C2.1, C3.2, C4.1, C5.2, R5.1, R7.2, U1.4 (GND), U1.7 (WP), U2.4 (GND), U3.2 (A1), U3.4 (GND), U3.7 (WP), U4.21 (GND), U4.3 (GND), U4.5 (GND)
- new net MISO: U4.16 (PB4)
- new net MOSI: U4.15 (PB3)
- new net RESET: R6.1, U4.29 (PC6/~{RESET})
- new net RX: U4.30 (PD0)
- new net TX: U4.31 (PD1)
- no-connect marks 0 -> 8
Other:
- added sheet Connectors (Connectors.kicad_sch)
- title: (none) -> ${project_name}
